Commit message: load tennis court maps && mini

File: tennisbuddy/description/urdf/mini.urdf (robot description, URDF)
Before this commit: robot rover_mini, 6 links, 5 joints
Links:
- link chassis_link: geometry collision mesh filename=file://$(find tennisbuddy_description)/meshes/mini_chassis_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; visual mesh filename=file://$(find tennisbuddy_description)/meshes/mini_chassis_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
- link fl_wheel_link: geometry collision mesh filename=file://$(find tennisbuddy_description)/meshes/65wheels.dae; visual mesh filename=file://$(find tennisbuddy_description)/meshes/65wheels.dae
- link fr_wheel_link: geometry collision mesh filename=file://$(find tennisbuddy_description)/meshes/65wheels.dae; visual mesh filename=file://$(find tennisbuddy_description)/meshes/65wheels.dae
- link rl_wheel_link: geometry collision mesh filename=file://$(find tennisbuddy_description)/meshes/65wheels.dae; visual mesh filename=file://$(find tennisbuddy_description)/meshes/65wheels.dae
- link rr_wheel_link: geometry collision mesh filename=file://$(find tennisbuddy_description)/meshes/65wheels.dae; visual mesh filename=file://$(find tennisbuddy_description)/meshes/65wheels.dae
