Commit message: planning

File: tennisbuddy/description/urdf/accessories/realsense_camera.urdf (robot description, URDF)
Before this commit: robot realsense_camera, 5 links, 5 joints
Joints:
- joint camera_to_payload: origin xyz=0.15 0.0 0.05 rpy=0 0 0 -> xyz=0.25 0.0 0.15 rpy=0 0 0; parent payload_link -> base_link
