Commit message: readme

File: tennisbuddy/description/urdf/accessories/imu.urdf (robot description, URDF)
Before this commit: robot imu, 1 links, 1 joints
Joints:
- removed joint imu_to_payload
- added joint imu_to_chassis: type fixed, parent chassis_link, child imu_link, origin xyz=0.0 0.0 0.21 rpy=0 0 0

File: tennisbuddy/description/urdf/accessories/realsense_camera.urdf (robot description, URDF)
Before this commit: robot realsense_camera, 5 links, 5 joints
Joints:
- removed joint camera_to_payload
- added joint camera_to_chassis: type fixed, parent chassis_link, child camera_link, origin xyz=0.25 0.0 0.15 rpy=0 0 0

File: tennisbuddy/description/urdf/accessories/rplidar_s2.urdf (robot description, URDF)
Before this commit: robot rplidar_s2, 1 links, 1 joints
Joints:
- removed joint lidar_to_payload
- added joint lidar_to_chassis: type fixed, parent chassis_link, child lidar_link, origin xyz=0.0 0 0.18 rpy=0 0 3.1415
